File: LM399_voltage_reference.kicad_sch (KiCad schematic)
At the start: 12 parts, among them U1 LM399, U2 LTC2057

Commit message: Done?
Parts:
- added H1, H2, H3, H4: MountingHole, MountingHole:MountingHole_3.2mm_M3, symbol Mechanical:MountingHole
Other:
- moved on the sheet: C1, C2, C3, C4, R1, RN1, TP1, TP2, TP3, TP4, U1, U2
